Commit message: 修改天工相关的代码与参数,支持控制四指

File: dextrah_lab/assets/tiangong/tiangong2pro.urdf (robot description, URDF)
Before this commit: robot tiangong2pro, 35 links, 34 joints
Links:
- link base_link_r: geometry collision box size=0.05 0.0674 0.15; visual mesh filename=meshes/base_link_r.STL
Joints:
- joint Joint_A01_R: limit lower=0.0 upper=1.5708 effort=0.05 velocity=7.5398223686155035 -> lower=0.0 upper=1.2217 effort=0.05 velocity=7.5398223686155035
- joint Joint_A02_R: limit lower=0.0 upper=1.5708 effort=0.05 velocity=7.5398223686155035 -> lower=0.0 upper=1.2217 effort=0.05 velocity=7.5398223686155035; mimic (none) -> joint=Joint_A01_R multiplier=1.0 offset=0.0; type fixed -> revolute
- joint Joint_B01_R: limit lower=0.0 upper=1.5708 effort=0.05 velocity=7.5398223686155035 -> lower=0.0 upper=1.2217 effort=0.05 velocity=7.5398223686155035
- joint Joint_B02_R: limit lower=0.0 upper=1.5708 effort=0.05 velocity=7.5398223686155035 -> lower=0.0 upper=1.2217 effort=0.05 velocity=7.5398223686155035; mimic (none) -> joint=Joint_B01_R multiplier=1.0 offset=0.0; type fixed -> revolute
- joint Joint_C01_R: limit lower=-0.0 upper=1.0 effort=0.05 velocity=7.5398223686155035 -> lower=-0.0 upper=1.2217 effort=0.05 velocity=7.5398223686155035; type fixed -> revolute
- joint Joint_C02_R: limit lower=0.0 upper=1.5708 effort=0.05 velocity=7.5398223686155035 -> lower=0.0 upper=1.2217 effort=0.05 velocity=7.5398223686155035; mimic (none) -> joint=Joint_C01_R multiplier=1.0 offset=0.0; type fixed -> revolute
- joint Joint_D01_R: limit lower=0.0 upper=1.0 effort=0.05 velocity=7.5398223686155035 -> lower=0.0 upper=1.2217 effort=0.05 velocity=7.5398223686155035; type fixed -> revolute
- joint Joint_D02_R: limit lower=0.0 upper=1.5708 effort=0.05 velocity=7.5398223686155035 -> lower=0.0 upper=1.2217 effort=0.05 velocity=7.5398223686155035; mimic (none) -> joint=Joint_D01_R multiplier=1.0 offset=0.0; type fixed -> revolute

Commit message: 尝试使用四指，运行不成功

File: dextrah_lab/assets/tiangong/tiangong2pro.urdf (robot description, URDF)
Before this commit: robot tiangong2pro, 35 links, 34 joints
Joints:
- joint Joint_A02_R: type revolute -> fixed
- joint Joint_B02_R: type revolute -> fixed
- joint Joint_C02_R: type revolute -> fixed
- joint Joint_D02_R: type revolute -> fixed
